File: UTv0/UTv0.kicad_sch (KiCad schematic)
At the start: 0 parts

Commit message: Transmit Circuit
Other:
- sheet Receive ports: added AnalogRx; removed none
- sheet Transmit ports: added Trig; removed none
Changed lines of the file:
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@@
 		(comment 4 "Stanford University")
+	)
+	(wire
+		(pts
+			(xy 124.46 132.08) (xy 133.35 132.08)
+		)
+		(stroke
+			(width 0)
+			(type default)
+		)
+	)
+	(wire
+		(pts
+			(xy 124.46 93.98) (xy 133.35 93.98)
+		)
+		(stroke
+			(width 0)
+			(type default)
+		)
 	)
 	(sheet
@@
 				)
 				(justify left top)
+			)
+		)
+		(pin "AnalogRx" output
+			(at 133.35 132.08 180)
+			(effects
+				(font
+					(size 1.27 1.27)
+				)
+				(justify left)
 			)
 		)
@@
 			)
 		)
+		(pin "Trig" input
+			(at 133.35 93.98 180)
+			(effects
+				(font
+					(size 1.27 1.27)
+				)
+				(justify left)
+			)
+		)
